File: ALPS-V1.kicad_pcb (KiCad board)
At the start: 2 copper layers, 118 x 45.5 mm, 13 parts, among them U1 LM317_TO-220

Commit message: Changed the label for the 5k potentiometer
Parts:
- renumbered Heavy to Coarse
Changed lines of the file:
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@@
 		(layer "F.Cu")
 		(at 139 95 -90)
-		(property "Reference" "Heavy"
+		(property "Reference" "Coarse"
 			(at -8.5 -8.5 180)
 			(layer "F.SilkS")
